Commit message: update joint limits

File: urdf/doodlebot.urdf (robot description, URDF)
Before this commit: robot doodlebot, 8 links, 7 joints
Joints:
- joint joint1: limit lower=-2.827433388230814 upper=2.827433388230814 effort=1 velocity=4.8 -> lower=-1.5707963267948966 upper=1.5707963267948966 effort=1 velocity=4.8
- joint joint2: limit lower=-1.790707812546182 upper=1.5707963267948966 effort=1 velocity=4.8 -> lower=-1.5707963267948966 upper=1.5707963267948966 effort=1 velocity=4.8
- joint joint3: limit lower=-0.9424777960769379 upper=1.382300767579509 effort=1 velocity=4.8 -> lower=-1.5707963267948966 upper=1.5707963267948966 effort=1 velocity=4.8
- joint joint4: limit lower=-1.790707812546182 upper=2.0420352248333655 effort=1 velocity=4.8 -> lower=-1.5707963267948966 upper=1.5707963267948966 effort=1 velocity=4.8

File: urdf/doodlebot.urdf.xacro (robot description, xacro)
@@ -31,5 +31,5 @@
     <origin xyz="0.0 0.0 0.0" rpy="0 0 0"/>
     <axis xyz="0 0 1"/>
-    <limit velocity="4.8" effort="1" lower="${-pi*0.9}" upper="${pi*0.9}" />
+    <limit velocity="4.8" effort="1" lower="${-pi*0.5}" upper="${pi*0.5}" />
   </joint>
   <!--  Link 2 -->
@@ -62,5 +62,5 @@
     <origin xyz="0.0 0.0 0.072475" rpy="0 0 0"/>
     <axis xyz="0 1 0"/>
-    <limit velocity="4.8" effort="1" lower="${-pi*0.57}" upper="${pi*0.5}" />
+    <limit velocity="4.8" effort="1" lower="${-pi*0.5}" upper="${pi*0.5}" />
   </joint>
   <!--  Link 3 -->
@@ -93,5 +93,5 @@
     <origin xyz="0.033335 0 0.135" rpy="0 0 0"/>
     <axis xyz="0 1 0"/>
-    <limit velocity="4.8" effort="1" lower="${-pi*0.3}" upper="${pi*0.44}" />
+    <limit velocity="4.8" effort="1" lower="${-pi*0.5}" upper="${pi*0.5}" />
   </joint>
   <!--  Link 4 -->
@@ -124,5 +124,5 @@
     <origin xyz="0.140 0.0 0.0" rpy="0 0 0"/>
     <axis xyz="0 1 0"/>
-    <limit velocity="4.8" effort="1" lower="${-pi*0.57}" upper="${pi*0.65}" />
+    <limit velocity="4.8" effort="1" lower="${-pi*0.5}" upper="${pi*0.5}" />
   </joint>
   <!--  Link 5 -->
